File: PCB/kraky_lite.kicad_sch (KiCad schematic)
At the start: 24 parts, among them J1 cc1101, J2 nfr24, J3 cc1101, J4 nfr24, J5 PINHD_1x7_Female, J7 2345986-1, SW1 Push_Button, SW2 Push_Button, SW3 Push_Button, SW4 Push_Button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

Commit message: Add files via upload
Parts:
- removed J5: PINHD_1x7_Female, Connector_PinSocket_2.54mm:PinSocket_1x07_P2.54mm_Vertical, symbol PCM_SL_Pin_Headers:PINHD_1x7_Female
- added J5: PINHD_1x8_Female, Connector_PinSocket_2.54mm:PinSocket_1x08_P2.54mm_Vertical, symbol PCM_SL_Pin_Headers:PINHD_1x8_Female
Connections:
- net GND: now also J5.8
- net at J1.4, J2.4, J3.4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: now also J5.6
- net at C1.2, C2.2, C3.2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: now also J5.1, J5.7
- net at U2.15 (IO3): now also J5.2
- net at J2.5, U2.18 (IO10): now also J5.5
- net at U2.38 (IO2): now also J5.3
- net at U2.39 (IO1): now also J5.4
